Commit message: add attach link plugin

File: robot_digital_twin/urdf/camera.xacro (robot description, xacro)
@@ -78,10 +78,10 @@
   <gazebo reference="link_camera_origin">
   <sensor name="$depth_camera" type="depth">
-    <update_rate>30</update_rate>
+    <update_rate>15</update_rate>
     <camera>
       <horizontal_fov>1.39626340156</horizontal_fov> <!-- 80deg -->
       <image>
-        <width>3840</width>
-        <height>2160</height>
+        <width>1920</width>
+        <height>1080</height>
         <format>R8G8B8</format>
       </image>

File: robot_digital_twin/urdf/gp4_wristcam.xacro (robot description, xacro)
@@ -391,5 +391,5 @@
                         color_width="1280"
                         color_height="720"
-                        color_fps="30"
+                        color_fps="15"
                         enable_pointCloud="true"
                         depth_width="1280"
@@ -406,5 +406,5 @@
                         color_width="1280"
                         color_height="720"
-                        color_fps="30"
+                        color_fps="15"
                         enable_pointCloud="true"
                         depth_width="1280"

File: robot_digital_twin/urdf/lego_2x4.xacro (robot description, xacro)
@@ -13,12 +13,12 @@
         rpy="0 0 0" />
       <mass
-        value="0.001" />
+        value="0.01" />
       <inertia
-        ixx="0"
+        ixx="0.0001"
         ixy="-0.0"
         ixz="0.0"
-        iyy="0.0"
+        iyy="0.0001"
         iyz="0.0"
-        izz="0.0" />
+        izz="0.0001" />
     </inertial>
     <visual>
@@ -36,5 +36,5 @@
       </material>
     </visual>
-    <!-- <collision>
+    <collision>
       <origin
         xyz="0 0 0"
@@ -44,9 +44,9 @@
           filename="file://$(find robot_digital_twin)/meshes/lego/b2x4.stl"/>
       </geometry>
-    </collision> -->
+    </collision>
     <gravity>0</gravity>
   </link>
   <gazebo reference="brick">
-  <kinematic>true</kinematic>
+  <!-- <kinematic>true</kinematic> -->
   <xacro:if value="${color == 'Orange'}">
      <material>Gazebo/Orange</material>

File: robot_digital_twin/urdf/lego_2x4（复件）.xacro (robot description, xacro)
@@ -1,11 +1,11 @@
 <?xml version="1.0" encoding="utf-8"?>
 <robot
-  name="base_plate48" xmlns:xacro="http://ros.org/wiki/xacro">
-  <xacro:macro name="base_plate48">
-  <xacro:arg name="plate_color" default="Orange" />
+  name="b2x4" xmlns:xacro="http://ros.org/wiki/xacro">
+  <xacro:macro name="b2x4">
+  <xacro:arg name="brick_color" default="Orange" />
   <xacro:property name="scale" value="0.001"/>
-  <xacro:property name="color" value="$(arg plate_color)"/>
+  <xacro:property name="color" value="$(arg brick_color)"/>
   <link
-    name="plate">
+    name="brick">
     <inertial>
       <origin
@@ -13,7 +13,7 @@
         rpy="0 0 0" />
       <mass
-        value="1" />
+        value="0.001" />
       <inertia
-        ixx="0"
+        ixx="0.0"
         ixy="-0.0"
         ixz="0.0"
@@ -25,8 +25,8 @@
       <origin
         xyz="0 0 0"
-        rpy="0 0 0" />
+        rpy="0 0 ${pi/2}" />
       <geometry>
         <mesh scale="${scale} ${scale} ${scale}"
-          filename="file://$(find robot_digital_twin)/meshes/lego/base48x48.stl"/>
+          filename="file://$(find robot_digital_twin)/meshes/lego/b2x4.stl"/>
       </geometry>
       <material
@@ -36,13 +36,16 @@
       </material>
     </visual>
-    <collision>
-      <origin xyz="0 0 -0.0025" rpy="0 0 0"/>
+    <!-- <collision>
+      <origin
+        xyz="0 0 0"
+        rpy="0 0 ${pi/2}" />
       <geometry>
-         <box size="0.48 0.48 0.005"/>
+        <mesh scale="${scale} ${scale} ${scale}"
+          filename="file://$(find robot_digital_twin)/meshes/lego/b2x4.stl"/>
       </geometry>
-    </collision>
+    </collision> -->
     <gravity>0</gravity>
   </link>
-  <gazebo reference="plate">
+  <gazebo reference="brick">
   <kinematic>true</kinematic>
   <xacro:if value="${color == 'Orange'}">
@@ -76,5 +79,5 @@
   </gazebo>
   </xacro:macro>
-  <xacro:base_plate48>
-  </xacro:base_plate48>
+  <xacro:b2x4>
+  </xacro:b2x4>
 </robot>

File: robot_digital_twin/urdf/lego_baseplate48（复件）.xacro (robot description, xacro)
@@ -13,5 +13,5 @@
         rpy="0 0 0" />
       <mass
-        value="1" />
+        value="0.001" />
       <inertia
         ixx="0"
@@ -36,10 +36,13 @@
       </material>
     </visual>
-    <collision>
-      <origin xyz="0 0 -0.0025" rpy="0 0 0"/>
+    <!-- <collision>
+      <origin
+        xyz="0 0 0"
+        rpy="0 0 0" />
       <geometry>
-         <box size="0.48 0.48 0.005"/>
+        <mesh scale="${scale} ${scale} ${scale}"
+          filename="file://$(find robot_digital_twin)/meshes/lego/base32x32.stl"/>
       </geometry>
-    </collision>
+    </collision> -->
     <gravity>0</gravity>
   </link>

Commit message: modify world setting

File: robot_digital_twin/urdf/camera.xacro (robot description, xacro)
@@ -77,11 +77,12 @@
   </xacro:camera>
   <gazebo reference="link_camera_origin">
-  <sensor name="$depth_camera" type="depth">
+  <!-- <sensor name="$depth_camera" type="depth">  -->
+  <sensor name="$depth_camera" type="camera">
     <update_rate>15</update_rate>
     <camera>
       <horizontal_fov>1.39626340156</horizontal_fov> <!-- 80deg -->
       <image>
-        <width>1920</width>
-        <height>1080</height>
+        <width>1280</width>
+        <height>720</height>
         <format>R8G8B8</format>
       </image>
@@ -91,5 +92,9 @@
       </clip>
     </camera>
-    <plugin name="$depth_camera_controller" filename="libgazebo_ros_openni_kinect.so">
+    <plugin name="rgb_camera_controller" filename="libgazebo_ros_camera.so">
+      <cameraName>fixed_camera</cameraName>
+      <frameName>depth_camera_link</frameName>
+    </plugin>
+    <!-- <plugin name="$depth_camera_controller" filename="libgazebo_ros_openni_kinect.so">
       <baseline>0.2</baseline>
       <alwaysOn>true</alwaysOn>
@@ -109,5 +114,5 @@
       <focalLength>0</focalLength>
       <hackBaseline>0</hackBaseline>
-    </plugin>
+    </plugin> -->
   </sensor>
 </gazebo>

File: robot_digital_twin/urdf/common_colours.xacro (robot description, xacro)
@@ -34,3 +34,4 @@
   <!-- not an official colour, but used in some old xacro:macros -->
   <xacro:property name="color_yaskawa_silver" value="0.8 0.8 0.8 1"/>
+  <xacro:property name="color_copper_red" value="${227/255} ${23/255} ${13/255} 1.0"/>
 </robot>

File: robot_digital_twin/urdf/common_materials.xacro (robot description, xacro)
@@ -95,3 +95,12 @@
     </material>
   </xacro:macro>
+  <xacro:macro name="tool_material_copper_red">
+    <material name="">
+        <color rgba="${color_copper_red}"/>
+        <ambient>0.4 0.4 0.4 1</ambient>
+        <diffuse>0.5 0.5 0.5 1</diffuse>
+        <specular>0.2 0.2 0.2 0</specular>
+        <emissive>0 0 0 1</emissive>
+    </material>
+  </xacro:macro>
 </robot>

File: robot_digital_twin/urdf/gp4_wristcam.xacro (robot description, xacro)
@@ -252,4 +252,5 @@
             <mesh filename="file://$(find robot_digital_twin)/meshes/eoat/tool_D405.stl"/>
           </geometry>
+          <xacro:tool_material_copper_red/>
         </visual>
         <!-- <collision>
@@ -392,5 +393,5 @@
                         color_height="720"
                         color_fps="15"
-                        enable_pointCloud="true"
+                        enable_pointCloud="false"
                         depth_width="1280"
                         depth_height="720"
@@ -407,5 +408,5 @@
                         color_height="720"
                         color_fps="15"
-                        enable_pointCloud="true"
+                        enable_pointCloud="false"
                         depth_width="1280"
                         depth_height="720"
@@ -447,5 +448,5 @@
   </gazebo>
   <gazebo reference="link_tool">
-     <material>Gazebo/Black</material>
+    <material>Gazebo/Orange</material>
     <visual> <transparency> 0 </transparency> </visual>
   </gazebo>

File: robot_digital_twin/urdf/lego_1x2_marker.xacro (robot description, xacro)
@@ -1,11 +1,11 @@
 <?xml version="1.0" encoding="utf-8"?>
 <robot
-  name="base_plate48" xmlns:xacro="http://ros.org/wiki/xacro">
-  <xacro:macro name="base_plate48">
-  <xacro:arg name="plate_color" default="Orange" />
+  name="b1x2" xmlns:xacro="http://ros.org/wiki/xacro">
+  <xacro:macro name="b1x2">
+  <xacro:arg name="brick_color" default="Orange" />
   <xacro:property name="scale" value="0.001"/>
-  <xacro:property name="color" value="$(arg plate_color)"/>
+  <xacro:property name="color" value="$(arg brick_color)"/>
   <link
-    name="plate">
+    name="brick">
     <inertial>
       <origin
@@ -24,9 +24,9 @@
     <visual>
       <origin
-        xyz="0 0 0"
-        rpy="0 0 0" />
+        xyz="0 0 0.002"
+        rpy="0 0 ${pi/2}" />
       <geometry>
         <mesh scale="${scale} ${scale} ${scale}"
-          filename="file://$(find robot_digital_twin)/meshes/lego/base48x48.stl"/>
+          filename="file://$(find robot_digital_twin)/meshes/lego/b1x2.stl"/>
       </geometry>
       <material
@@ -39,13 +39,13 @@
       <origin
         xyz="0 0 0"
-        rpy="0 0 0" />
+        rpy="0 0 ${pi/2}" />
       <geometry>
         <mesh scale="${scale} ${scale} ${scale}"
-          filename="file://$(find robot_digital_twin)/meshes/lego/base32x32.stl"/>
+          filename="file://$(find robot_digital_twin)/meshes/lego/b1x2.stl"/>
       </geometry>
     </collision> -->
     <gravity>0</gravity>
   </link>
-  <gazebo reference="plate">
+  <gazebo reference="brick">
   <kinematic>true</kinematic>
   <xacro:if value="${color == 'Orange'}">
@@ -76,8 +76,8 @@
      <material>Gazebo/Purple</material>
     </xacro:if>
-    <visual> <transparency> 0 </transparency> </visual>
+    <visual> <transparency> 0.5 </transparency> </visual>
   </gazebo>
   </xacro:macro>
-  <xacro:base_plate48>
-  </xacro:base_plate48>
+  <xacro:b1x2>
+  </xacro:b1x2>
 </robot>

File: robot_digital_twin/urdf/lego_2x4.xacro (robot description, xacro)
@@ -4,6 +4,8 @@
   <xacro:macro name="b2x4">
   <xacro:arg name="brick_color" default="Orange" />
+  <xacro:arg name="physics" default="false"/>
   <xacro:property name="scale" value="0.001"/>
   <xacro:property name="color" value="$(arg brick_color)"/>
+  <xacro:property name="physics" value="$(arg physics)"/>
   <link
     name="brick">
@@ -36,17 +38,21 @@
       </material>
     </visual>
-    <collision>
-      <origin
-        xyz="0 0 0"
-        rpy="0 0 ${pi/2}" />
-      <geometry>
-        <mesh scale="${scale} ${scale} ${scale}"
-          filename="file://$(find robot_digital_twin)/meshes/lego/b2x4.stl"/>
-      </geometry>
-    </collision>
+    <xacro:if value="${physics}">
+      <collision>
+        <origin
+          xyz="0 0 0"
+          rpy="0 0 ${pi/2}" />
+        <geometry>
+          <mesh scale="${scale} ${scale} ${scale}"
+            filename="file://$(find robot_digital_twin)/meshes/lego/b2x4.stl"/>
+        </geometry>
+      </collision>
+    </xacro:if>
     <gravity>0</gravity>
   </link>
   <gazebo reference="brick">
-  <!-- <kinematic>true</kinematic> -->
+  <xacro:if value="${not physics}">
+    <kinematic>true</kinematic>
+  </xacro:if>
   <xacro:if value="${color == 'Orange'}">
      <material>Gazebo/Orange</material>

File: robot_digital_twin/urdf/lego_baseplate48.xacro (robot description, xacro)
@@ -4,6 +4,8 @@
   <xacro:macro name="base_plate48">
   <xacro:arg name="plate_color" default="Orange" />
+  <xacro:arg name="physics" default="false"/>
   <xacro:property name="scale" value="0.001"/>
   <xacro:property name="color" value="$(arg plate_color)"/>
+  <xacro:property name="physics" value="$(arg physics)"/>
   <link
     name="plate">
@@ -13,5 +15,5 @@
         rpy="0 0 0" />
       <mass
-        value="1" />
+        value="0.001" />
       <inertia
         ixx="0"
@@ -36,42 +38,46 @@
       </material>
     </visual>
-    <collision>
-      <origin xyz="0 0 -0.0025" rpy="0 0 0"/>
-      <geometry>
-         <box size="0.48 0.48 0.005"/>
-      </geometry>
-    </collision>
+    <xacro:if value="${physics}">
+      <collision>
+        <origin xyz="0 0 -0.0025" rpy="0 0 0"/>
+        <geometry>
+          <box size="0.48 0.48 0.005"/>
+        </geometry>
+      </collision>
+    </xacro:if>
     <gravity>0</gravity>
   </link>
   <gazebo reference="plate">
-  <kinematic>true</kinematic>
-  <xacro:if value="${color == 'Orange'}">
-     <material>Gazebo/Orange</material>
-    </xacro:if>
-    <xacro:if value="${color == 'Green'}">
-     <material>Gazebo/Green</material>
-    </xacro:if>
-    <xacro:if value="${color == 'Black'}">
-     <material>Gazebo/Black</material>
-    </xacro:if>
-    <xacro:if value="${color == 'Blue'}">
-     <material>Gazebo/Blue</material>
-     </xacro:if>
-     <xacro:if value="${color == 'Yellow'}">
-     <material>Gazebo/Yellow</material>
-    </xacro:if>
-    <xacro:if value="${color == 'Red'}">
-     <material>Gazebo/Red</material>
-    </xacro:if>
-    <xacro:if value="${color == 'White'}">
-     <material>Gazebo/White</material>
-    </xacro:if>
-    <xacro:if value="${color == 'Grey'}">
-     <material>Gazebo/Grey</material>
-    </xacro:if>
-    <xacro:if value="${color == 'Purple'}">
-     <material>Gazebo/Purple</material>
-    </xacro:if>
-    <visual> <transparency> 0 </transparency> </visual>
+    <!-- <xacro:if value="${not physics}"> -->
+      <kinematic>true</kinematic>
+    <!-- </xacro:if> -->
+    <xacro:if value="${color == 'Orange'}">
+       <material>Gazebo/Orange</material>
+      </xacro:if>
+      <xacro:if value="${color == 'Green'}">
+       <material>Gazebo/Green</material>
+      </xacro:if>
+      <xacro:if value="${color == 'Black'}">
+       <material>Gazebo/Black</material>
+      </xacro:if>
+      <xacro:if value="${color == 'Blue'}">
+       <material>Gazebo/Blue</material>
+       </xacro:if>
+       <xacro:if value="${color == 'Yellow'}">
+       <material>Gazebo/Yellow</material>
+      </xacro:if>
+      <xacro:if value="${color == 'Red'}">
+       <material>Gazebo/Red</material>
+      </xacro:if>
+      <xacro:if value="${color == 'White'}">
+       <material>Gazebo/White</material>
+      </xacro:if>
+      <xacro:if value="${color == 'Grey'}">
+       <material>Gazebo/Grey</material>
+      </xacro:if>
+      <xacro:if value="${color == 'Purple'}">
+       <material>Gazebo/Purple</material>
+      </xacro:if>
+      <visual> <transparency> 0 </transparency> </visual>
   </gazebo>
   </xacro:macro>
